File: hardware/Victor9K_pga2350.kicad_sch (KiCad schematic)
At the start: 23 parts, among them IC1 74LVC1G14GW,125, J1 PICO DEBUG, J2 Micro_SD_Card, J4 DX07S016JA1R1500, J5 UART, SW1 BOOTSEL, U1 ESP32-S3-DevKitC

Commit message: reworked PCB for latest gpio configuration. added reset connect to 8088, adjusted SIP for SD card instead of SDIO. added UART RX and SIP breakout pins.
Parts:
- removed C13, C8: 0.1µF, Capacitor_THT:C_Disc_D5.0mm_W2.5mm_P5.00mm, symbol Device:C
- removed IC1: 74LVC1G14GW,125, Victor9000:SOT65P212X110-5N, symbol Victor9K_symbols:74LVC1G14GW,125
- removed U1: ESP32-S3-DevKitC, Victor9000:ESP32-S3-DevKitC, symbol Espressif-2:ESP32-S3-DevKitC
- added D1, D2: 1N4148, Diode_THT:D_DO-35_SOD27_P7.62mm_Horizontal, symbol Diode:1N4148
- added IC1: SN74LVC1G04QDCKRQ1, Victor9000:SOT65P210X110-5N, symbol Victor9K_symbols:SN74LVC1G04QDCKRQ1
- added J2: SPI Breakout, Connector_PinHeader_2.54mm:PinHeader_1x06_P2.54mm_Vertical, symbol Connector:Conn_01x06_Pin
- added R3: 470Ω, Resistor_THT:R_Axial_DIN0204_L3.6mm_D1.6mm_P5.08mm_Horizontal, symbol Device:R
- added R4: 2.2KΩ, Resistor_THT:R_Axial_DIN0204_L3.6mm_D1.6mm_P5.08mm_Horizontal, symbol Device:R
- added RN1: 47KΩ, 4609X101473LF, symbol Victor9K_symbols:4609X-101-473LF
- added RN2: 2.7KΩ, Resistor_THT:R_Array_SIP4, symbol Device:R_Network03
- C3: value 0.1µF -> 1µF
- C7: value 0.1µF -> .01µF
- J4: value DX07S016JA1R1500 -> USB C DX07S016JA1R1500
- Jd1: renamed from J2; footprint Victor9000:DM3ATSFPEJM5 -> Victor9000:HRS_DM3AT-SF-PEJM5; symbol Connector:Micro_SD_Card -> Victor9K_symbols:DM3AT-SF-PEJM5; MAXIMUM_PACKAGE_HEIGHT (none) -> 1.83 mm; MF (none) -> Hirose Electric Co Ltd; MP (none) -> DM3AT-SF-PEJM5; PARTREV (none) -> 20200913
Connections:
- net FN_CS is gone; now on net SD_CS: A1.41 (GPIO41)
- net FN_INT is gone; now on net SD_MISO: A1.44 (GPIO44)
- net FN_MISO is gone; now on net DEN: A1.40 (GPIO40)
- net FN_MOSI is gone; now on net SD_MOSI: A1.43 (GPIO43)
- net FN_SCLK is gone; now on net SD_SCLK: A1.42 (GPIO42)
- net +3.3V: now also IC1.5 (VCC), RN1.1
- net +5V: now also R3.1, RN2.1 (common); no longer C7.1
- net ALE: now also D1.1 (K), R4.1
- net DEN: no longer A1.25 (GPIO25)
- net DT/R: now also RN2.2 (R1)
- net GND: now also Jd1.P1 (SHIELD), Jd1.P2 (SHIELD), Jd1.P3 (SHIELD), Jd1.P4 (SHIELD), D2.1 (K), IC1.3 (GND)
- net HOLD: now also A1.25 (GPIO25); no longer A1.26 (GPIO26)
- net IO/M: now also A1.35 (GPIO35); no longer A1.34 (GPIO34)
- net IR5: now also A1.34 (GPIO34); no longer A1.35 (GPIO35)
- net RD: now also RN2.4 (R3)
- net RESET: now also IC1.2 (A)
- net SD_CS: now also J2.1 (Pin_1), RN1.3
- net SD_MISO: now also Jd1.7 (DAT0), J2.4 (Pin_4), RN1.7; no longer Jd1.3 (CMD)
- net SD_MOSI: now also Jd1.3 (CMD), J2.3 (Pin_3), RN1.4; no longer Jd1.7 (DAT0)
- net SD_SCLK: now also J2.2 (Pin_2), RN1.5
- net UART RX: now also A1.33 (GPIO33); no longer A1.46 (GPIO46)
- net WR: now also RN2.3 (R2)
- net XACK: now also A1.26 (GPIO26); no longer A1.33 (GPIO33)
- net SD_DAT2: now reaches Jd1.1 (DAT2)
- net SD_DAT2: now also RN1.2
- net SD_DAT1: now reaches Jd1.8 (DAT1)
- net SD_DAT1: now also RN1.8
- net GPIO45: now reaches A1.45 (GPIO45)
- net GPIO45: now also J2.5 (Pin_5)
- net -12VLT renamed -12V
- net -12V: now also C7.1, R4.2
- net NOT_RESET renamed RUN
- net RUN: now also IC1.4 (Y)
- new net: D1.2 (A), D2.2 (A), R3.2
- new net GPIO46: A1.46 (GPIO46), J2.6 (Pin_6)
Other:
- note added: "26-Apr-2026"
- note added: "ALE Constant Current Pulldown Network"
- note added: "Control Sig Resistor Network"
- note added: "SD Card Resistor Network"
- note removed: "14-Apr-2025"
- moved on the sheet: A1, C1, C10, C11, C12, C2, C3, C4, C5, J1, J4, J5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
