File: hardware/rev2/v9k_dma_rev2.kicad_sch (KiCad schematic)
At the start: 38 parts, among them IC1 SN74LVC1G04, J10 EXPANDER GPIO, J3 microSD, J4 OLED SPI, J5 ENCODER, J6 ACT LED, J7 ESP32 BREAKOUT, J8 DEBUG UART, J9 SWD, U1 WeAct RP2350B Core, U3 ESP32-S3-WROOM-1U-N16R8, U4 LD1117V33, U5 MCP23S17

Commit message: v9k_dma_rev2: complete stages 4-6 — placed, routed (ROUTE OK), BOM finalized
- Placement + routing via llm_autoroute (margin-1 sweep winner): 122/122 nets,
  4940mm track, 252 vias, GND pours ~60% both layers, 0 unrouted, 0 hard DRC
  (kicad-cli verified; 68 cosmetic silk items remain). R3/R4/C8 moved clear of
  the USB-C plug path per review.
- U3 WROOM thermal vias enlarged to 0.3mm drill (board min-hole conflict);
  J3 edge-mount microSD edge-clearance exemption via v9k_dma_rev2.kicad_dru.
- Schematic: MPN fields populated from project.toml [[parts]] (19 symbols);
  U1/GF1 excluded from BOM (own stock / PCB feature).
- Stage 6: check-bom 0 errors, order_bom.csv $107.23 for 5 boards
  (DK $102.57 + Mouser $4.66); shunts for JP1/JP2 + 5x WeAct module are
  manual offsets.
- project.toml stage = 6 (all gates passed); skill_feedback.md items 14-25.
- .gitignore: llm_autoroute transient artifacts (pre-* backups, sweep logs).

Co-Authored-By: Claude Fable 5 <noreply@anthropic.com>
Parts:
- C11, C5, C7, C9: MPN (none) -> RD20B104K500A5HAND
- C2, C3, C4, C8: MPN (none) -> 50YXJ10M5X11
- D2, D3: MPN (none) -> 1N4148
- GF1, U1: now left out of the parts list
- J10, J4, J5, J6, J7, J8, J9, JP1, JP2: MPN (none) -> PREC040SAAN-RC

Commit message: rev2: adopt machine-readable source keys; GF1 MPN via set-part-fields
- project.toml: source = "stock" (U1) / "pcb-feature" (GF1) per the
  PROJECT_TOML.md convention, replacing the comment-only grouping — the new
  edablock set-part-fields / lint-sch check_mpn key off it.
- Schematic: GF1 MPN property stamped by set-part-fields (validation run of
  the new tool against this project; lint-sch exits 0).

Co-Authored-By: Claude Fable 5 <noreply@anthropic.com>
Parts:
- GF1: MPN (none) -> Victor gold fingers
Changed lines of the file:
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@@
       (effects (font (size 1.27 1.27)) hide)
+    )
+    (property "MPN" "Victor gold fingers" (id 5) (at 71.12 180.34 0)
+      (effects (font (size 1.0 1.0)) hide)
     )
     (instances
